Commit message: everything is working fine

File: urdf/robot.urdf (robot description, URDF)
Before this commit: robot arm, 8 links, 7 joints
Links:
- link base_1: mass None -> 1.0
- link end_effector_link: mass None -> 0.1; geometry collision box size=0.05 0.01 0.01; visual box size=0.05 0.01 0.01
- link forearm_link: mass None -> 1.0; geometry collision cylinder length=0.07 radius=0.03; visual cylinder length=0.07 radius=0.03
- link shoulder_link: mass None -> 1.0; geometry collision cylinder length=0.35 radius=0.03; visual cylinder length=0.35 radius=0.03
- link upper_arm_link: mass None -> 1.0; geometry collision cylinder length=0.35 radius=0.03; visual cylinder length=0.35 radius=0.03
- link wrist_1_link: mass None -> 1.0; geometry collision cylinder length=0.1 radius=0.03; visual cylinder length=0.1 radius=0.03
- link wrist_2_link: mass None -> 1.0; geometry collision cylinder length=0.05 radius=0.03; visual cylinder length=0.05 radius=0.03
Joints:
- removed joint base
- removed joint base_shoulder
- added joint base_1_shoulder: type revolute, parent base_1, child shoulder_link, origin xyz=0.0 0 0.135 rpy=0 0 0, axis 1 0 0, limit lower=-1.57 upper=1.57 effort=1000 velocity=10
- added joint base_base_1: type revolute, parent base_link, child base_1, origin xyz=0.0 0 0.005 rpy=0 0 0, axis 0 0 1, limit lower=-3.14 upper=3.14 effort=1000 velocity=10
- joint forearm_wrist_1: limit lower=-3.14159265359 upper=3.14159265359 effort=1000 velocity=10 -> lower=-1.57 upper=1.57 effort=1000 velocity=10; origin xyz=0.065 0 0 rpy=0 0 0 -> xyz=0.065 0 0.03 rpy=0 0 0
- joint shoulder_upper_arm: limit lower=-3.14159265359 upper=3.14159265359 effort=1000 velocity=10 -> lower=-1.57 upper=1.57 effort=1000 velocity=10; origin xyz=0.0 0 0.34 rpy=0 0 0 -> xyz=0.0 0 0.32 rpy=0 0 0
- joint upper_arm_forearm: limit lower=-3.14159265359 upper=3.14159265359 effort=1000 velocity=10 -> lower=-1.57 upper=1.57 effort=1000 velocity=10; origin xyz=0.0 0 0.32 rpy=0 0 0 -> xyz=0.0 0 0.305 rpy=0 0 0
- joint wrist_1_wrist_2: limit lower=-3.14159265359 upper=3.14159265359 effort=1000 velocity=10 -> lower=-1.57 upper=1.57 effort=1000 velocity=10; origin xyz=0.0 0 0.10 rpy=0 0 0 -> xyz=0.03 0 0.073 rpy=0 0 0
- joint wrist_2_end_effector: origin xyz=0.08 0 0 rpy=0 0 0 -> xyz=0.081 0 0 rpy=0 0 0

File: urdf/robot.urdf.xacro (robot description, xacro)
@@ -1,9 +1,13 @@
 <?xml version="1.0"?>
 <robot name="arm" xmlns:xacro="http://www.ros.org/wiki/xacro">
+    <xacro:include filename="gripper.urdf.xacro"/>
+    <material name="grey">
+        <color rgba="0.5 0.5 0.5 1" />
+    </material>
     <link name="base_link">
         <visual>
             <origin xyz="0 0 0" rpy="0 0 0" />
             <geometry>
-                <box size="0.5 0.5 0.01" />
+                <box size="0.25 0.25 0.01" />
             </geometry>
             <material name="grey">
@@ -14,188 +18,229 @@
             <origin xyz="0 0 0" rpy="0 0 0" />
             <geometry>
-                <box size="0.5 0.5 0.01" />
-            </geometry>
-        </collision>
-    </link>
-    <joint name="base" type="revolute">
+                <box size="0.20 0.20 0.005" />
+            </geometry>
+        </collision>
+    </link>
+    <joint name="base_base_1" type="revolute">
         <parent link="base_link"/>
         <child link="base_1"/>
-        <origin xyz="0.0 0 0.0" rpy="0 0 0"/>
+        <origin xyz="0.0 0 0.005" rpy="0 0 0"/>
         <axis xyz="0 0 1"/>
         <limit effort="1000" lower="-3.14" upper="3.14" velocity="10"/>
     </joint>
-    <joint name="base_shoulder" type="revolute">
+    <link name="base_1">
+        <visual>
+            <origin xyz="0 0 0.075" rpy="0 0 0"/>
+            <geometry>
+                <cylinder radius="0.03" length="0.15"/>
+            </geometry>
+            <material name="grey"/>
+        </visual>
+        <collision>
+            <origin xyz="0 0 0.075" rpy="0 0 0"/>
+            <geometry>
+                <cylinder radius="0.025" length="0.10"/>
+            </geometry>
+        </collision>
+        <inertial>
+            <origin xyz="0 0 0.075" rpy="0 0 0"/>
+            <mass value="1.0"/>
+            <inertia ixx="0.01" ixy="0" ixz="0" iyy="0.01" iyz="0" izz="0.01"/>
+        </inertial>
+    </link>
+    <joint name="base_1_shoulder" type="revolute">
         <parent link="base_1"/>
         <child link="shoulder_link"/>
-        <origin xyz="0.0 0 0.15" rpy="0 0 0"/>
-        <axis xyz="1 0 0"/>
-        <limit effort="1000" lower="-1.57" upper="1.57" velocity="10"/>
-    </joint >
+        <origin xyz="0.0 0 0.135" rpy="0 0 0"/>
+        <axis xyz="1 0 0"/>
+        <limit effort="1000" lower="-1.57" upper="1.57" velocity="10"/>
+    </joint>
+    <link name="shoulder_link">
+        <visual>
+            <origin xyz="0.063 0 0.160" rpy="0 0 0"/>
+            <geometry>
+                <cylinder radius="0.03" length="0.35"/>
+            </geometry>
+            <material name="grey"/>
+        </visual>
+        <collision>
+            <origin xyz="0.063 0 0.160" rpy="0 0 0"/>
+            <geometry>
+                <cylinder radius="0.025" length="0.30"/>
+            </geometry>
+        </collision>
+        <inertial>
+            <origin xyz="0.063 0 0.160" rpy="0 0 0"/>
+            <mass value="1.0"/>
+            <inertia ixx="0.01" ixy="0" ixz="0" iyy="0.01" iyz="0" izz="0.01"/>
+        </inertial>
+    </link>
     <joint name="shoulder_upper_arm" type="revolute">
         <parent link="shoulder_link"/>
         <child link="upper_arm_link"/>
-        <origin xyz="0.0 0 0.34" rpy="0 0 0"/>
-        <axis xyz="1 0 0"/>
-        <limit effort="1000" lower="-1.57" upper="1.57" velocity="10"/>
-    </joint>
+        <origin xyz="0.0 0 0.32" rpy="0 0 0"/>
+        <axis xyz="1 0 0"/>
+        <limit effort="1000" lower="-1.57" upper="1.57" velocity="10"/>
+    </joint>
+    <link name="upper_arm_link">
+        <visual>
+            <origin xyz="0.0 0 0.160" rpy="0 0 0"/>
+            <geometry>
+                <cylinder radius="0.03" length="0.35"/>
+            </geometry>
+            <material name="grey"/>
+        </visual>
+        <collision>
+            <origin xyz="0.0 0 0.160" rpy="0 0 0"/>
+            <geometry>
+                <cylinder radius="0.025" length="0.30"/>
+            </geometry>
+        </collision>
+        <inertial>
+            <origin xyz="0.0 0 0.160" rpy="0 0 0"/>
+            <mass value="1.0"/>
+            <inertia ixx="0.01" ixy="0" ixz="0" iyy="0.01" iyz="0" izz="0.01"/>
+        </inertial>
+    </link>
     <joint name="upper_arm_forearm" type="revolute">
         <parent link="upper_arm_link"/>
         <child link="forearm_link"/>
-        <origin xyz="0.0 0 0.32" rpy="0 0 0"/>
-        <axis xyz="1 0 0"/>
-        <limit effort="1000" lower="-1.57" upper="1.57" velocity="10"/>
-    </joint>
+        <origin xyz="0.0 0 0.305" rpy="0 0 0"/>
+        <axis xyz="1 0 0"/>
+        <limit effort="1000" lower="-1.57" upper="1.57" velocity="10"/>
+    </joint>
+    <link name="forearm_link">
+        <visual>
+            <origin xyz="0.068 0 0" rpy="0 1.57 0"/>
+            <geometry>
+                <cylinder radius="0.03" length="0.07"/>
+            </geometry>
+            <material name="grey"/>
+        </visual>
+        <collision>
+            <origin xyz="0.068 0 0" rpy="0 1.57 0"/>
+            <geometry>
+                <cylinder radius="0.025" length="0.06"/>
+            </geometry>
+        </collision>
+        <inertial>
+            <origin xyz="0.068 0 0" rpy="0 1.57 0"/>
+            <mass value="1.0"/>
+            <inertia ixx="0.01" ixy="0" ixz="0" iyy="0.01" iyz="0" izz="0.01"/>
+        </inertial>
+    </link>
     <joint name="forearm_wrist_1" type="revolute">
         <parent link="forearm_link"/>
         <child link="wrist_1_link"/>
-        <origin xyz="0.065 0 0" rpy="0 0 0"/>
+        <origin xyz="0.065 0 0.03" rpy="0 0 0"/>
         <axis xyz="0.0 0.0 1.0"/>
         <limit effort="1000" lower="-1.57" upper="1.57" velocity="10"/>
     </joint>
+    <link name="wrist_1_link">
+        <visual>
+            <origin xyz="0.0 0 0.053" rpy="0 0 0"/>
+            <geometry>
+                <cylinder radius="0.03" length="0.1"/>
+            </geometry>
+            <material name="grey"/>
+        </visual>
+        <collision>
+            <origin xyz="0.0 0 0.053" rpy="0 0 0"/>
+            <geometry>
+                <cylinder radius="0.025" length="0.09"/>
+            </geometry>
+        </collision>
+        <inertial>
+            <origin xyz="0.0 0 0.053" rpy="0 0 0"/>
+            <mass value="1.0"/>
+            <inertia ixx="0.01" ixy="0" ixz="0" iyy="0.01" iyz="0" izz="0.01"/>
+        </inertial>
+    </link>
     <joint name="wrist_1_wrist_2" type="revolute">
         <parent link="wrist_1_link"/>
         <child link="wrist_2_link"/>
-        <origin xyz="0.0 0 0.10" rpy="0 0 0"/>
-        <axis xyz="1 0 0"/>
-        <limit effort="1000" lower="-1.57" upper="1.57" velocity="10"/>
-    </joint>
+        <origin xyz="0.03 0 0.073" rpy="0 0 0"/>
+        <axis xyz="1 0 0"/>
+        <limit effort="1000" lower="-1.57" upper="1.57" velocity="10"/>
+    </joint>
+    <link name="wrist_2_link">
+        <visual>
+            <origin xyz="0.028 0.0 0.0" rpy="0 1.57 0" />
+            <geometry>
+                <cylinder radius="0.03" length="0.05"/>
+            </geometry>
+            <material name="grey"/>
+        </visual>
+        <collision>
+            <origin xyz="0.028 0.0 0.0" rpy="0 1.57 0" />
+            <geometry>
+                <cylinder radius="0.025" length="0.04"/>
+            </geometry>
+        </collision>
+        <inertial>
+            <origin xyz="0.028 0.0 0.0" rpy="0 1.57 0" />
+            <mass value="1.0"/>
+            <inertia ixx="0.01" ixy="0" ixz="0" iyy="0.01" iyz="0" izz="0.01"/>
+        </inertial>
+    </link>
     <joint name="wrist_2_end_effector" type="fixed">
         <parent link="wrist_2_link"/>
         <child link="end_effector_link"/>
-        <origin xyz="0.08 0 0" rpy="0 0 0"/>
-    </joint>
-    <link name="base_1">
-        <visual>
-            <origin xyz="0 0 0.08" rpy="0 0 0"/>
-            <geometry>
-                <cylinder radius="0.03" length="0.15"/>
-            </geometry>
-            <material name="grey">
-                <color rgba="0.5 0.5 0.5 1" />
-            </material>
-        </visual>
-        <collision>
-            <origin xyz="0 0 0.08" rpy="0 0 0"/>
-            <geometry>
-                <cylinder radius="0.03" length="0.15"/>
-            </geometry>
-        </collision>
-        <inertial>
-            <origin xyz="0 0 0.08" rpy="0 0 0"/>
-            <mass value="1.0"/>
-            <inertia ixx="0.01" ixy="0" ixz="0" iyy="0.01" iyz="0" izz="0.01"/>
-        </inertial>
-    </link>
-    <link name="shoulder_link">
-        <visual>
-            <origin xyz="0.06 0 0.175" rpy="0 0 0"/>
-            <geometry>
-                <cylinder radius="0.03" length="0.35"/>
-            </geometry>
-        </visual>
-        <collision>
-            <origin xyz="0.06 0 0.175" rpy="0 0 0"/>
-            <geometry>
-                <cylinder radius="0.03" length="0.35"/>
-            </geometry>
-        </collision>
-        <inertial>
-            <origin xyz="0.06 0 0.175" rpy="0 0 0"/>
-            <mass value="1.0"/>
-            <inertia ixx="0.01" ixy="0" ixz="0" iyy="0.01" iyz="0" izz="0.01"/>
-        </inertial>
-    </link>
-    <link name="upper_arm_link">
-        <visual>
-            <origin xyz="0.0 0 0.175" rpy="0 0 0"/>
-            <geometry>
-                <cylinder radius="0.03" length="0.35"/>
-            </geometry>
-            <material name="grey">
-                <color rgba="0.5 0.5 0.5 1" />
-            </material>
-        </visual>
-        <collision>
-            <origin xyz="0.0 0 0.175" rpy="0 0 0"/>
-            <geometry>
-                <cylinder radius="0.03" length="0.35"/>
-            </geometry>
-        </collision>
-        <inertial>
-            <origin xyz="0.0 0 0.175" rpy="0 0 0"/>
-            <mass value="1.0"/>
-            <inertia ixx="0.01" ixy="0" ixz="0" iyy="0.01" iyz="0" izz="0.01"/>
-        </inertial>
-    </link>
-    <link name="forearm_link">
-        <visual>
-            <origin xyz="0.065 0 0" rpy="0 1.57 0"/>
-            <geometry>
-                <cylinder radius="0.03" length="0.07"/>
-            </geometry>
-        </visual>
-        <collision>
-            <origin xyz="0.065 0 0" rpy="0 1.57 0"/>
-            <geometry>
-                <cylinder radius="0.03" length="0.07"/>
-            </geometry>
-        </collision>
-        <inertial>
-            <origin xyz="0.065 0 0" rpy="0 1.57 0"/>
-            <mass value="1.0"/>
-            <inertia ixx="0.01" ixy="0" ixz="0" iyy="0.01" iyz="0" izz="0.01"/>
-        </inertial>
-    </link>
-    <link name ="wrist_1_link">
-        <visual>
-            <origin xyz="0.0 0 0.08" rpy="0 0 0"/>
-            <geometry>
-                <cylinder radius="0.03" length="0.1"/>
-            </geometry>
-        </visual>
-        <collision>
-            <origin xyz="0.0 0 0.08" rpy="0 0 0"/>
-            <geometry>
-                <cylinder radius="0.03" length="0.1"/>
-            </geometry>
-        </collision>
-        <inertial>
-            <origin xyz="0.0 0 0.08" rpy="0 0 0"/>
-            <mass value="1.0"/>
-            <inertia ixx="0.01" ixy="0" ixz="0" iyy="0.01" iyz="0" izz="0.01"/>
-        </inertial>
-    </link>
-    <link name="wrist_2_link" >
-        <visual>
-            <origin xyz="0.055 0.0 0.0" rpy="0 1.57 0" />
-            <geometry>
-                <cylinder radius="0.03" length="0.05"/>
-            </geometry>
-            <collision>
-                <origin xyz="0.055 0.0 0.0" rpy="0 1.57 0" />
-                <geometry>
-                    <cylinder radius="0.03" length="0.05"/>
-                </geometry>
-            </collision>
-            <inertial>
-                <origin xyz="0.055 0.0 0.0" rpy="0 1.57 0" />
-                <mass value="1.0"/>
-                <inertia ixx="0.01" ixy="0" ixz="0" iyy="0.01" iyz="0" izz="0.01"/>
-            </inertial>
-        </visual>
-    </link>
+        <origin xyz="0.061 0 0" rpy="0 0 0"/>
+    </joint>
     <link name="end_effector_link">
         <visual>
-            <origin xyz="0.01 0 0" rpy="0 0 0" />
-            <geometry>
-                <box size="0.1 0.01 0.01"/>
-            </geometry>
-        </visual>
-        <collision>
-            <origin xyz="0.01 0 0" rpy="0 0 0" />
-            <geometry>
-                <box size="0.1 0.01 0.01"/>
-            </geometry>
-        </collision>
-    </link>
+            <origin xyz="0 0 0" rpy="0 0 0" />
+            <geometry>
+                <box size="0.01 0.01 0.01"/>
+            </geometry>
+            <material name="grey"/>
+        </visual>
+        <collision>
+            <origin xyz="0 0 0" rpy="0 0 0" />
+            <geometry>
+                <box size="0.005 0.005 0.005"/>
+            </geometry>
+        </collision>
+        <inertial>
+            <origin xyz="0 0 0" rpy="0 0 0"/>
+            <mass value="0.1"/>
+            <inertia ixx="0.0001" ixy="0" ixz="0" iyy="0.0001" iyz="0" izz="0.0001"/>
+        </inertial>
+    </link>
+    <ros2_control name="ArmHardware" type="system">
+      <hardware>
+        <plugin>fake_components/GenericSystem</plugin>
+      </hardware>
+      <joint name="base_base_1">
+        <command_interface name="position"/>
+        <state_interface name="position"/>
+        <state_interface name="velocity"/>
+      </joint>
+      <joint name="base_1_shoulder">
+        <command_interface name="position"/>
+        <state_interface name="position"/>
+        <state_interface name="velocity"/>
+      </joint>
+      <joint name="shoulder_upper_arm">
+        <command_interface name="position"/>
+        <state_interface name="position"/>
+        <state_interface name="velocity"/>
+      </joint>
+      <joint name="upper_arm_forearm">
+        <command_interface name="position"/>
+        <state_interface name="position"/>
+        <state_interface name="velocity"/>
+      </joint>
+      <joint name="forearm_wrist_1">
+        <command_interface name="position"/>
+        <state_interface name="position"/>
+        <state_interface name="velocity"/>
+      </joint>
+      <joint name="wrist_1_wrist_2">
+        <command_interface name="position"/>
+        <state_interface name="position"/>
+        <state_interface name="velocity"/>
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