Commit message: added gripper to urdf and made a single launch file for everything

File: urdf/gripper.urdf.xacro (robot description, xacro)
@@ -1,5 +1,11 @@
 <?xml version="1.0"?>
-<robot
-  name="gripper">
+<robot name="gripper">
+  <joint name="wrist_2_end_effector" type="revolute">
+    <origin xyz="0.061 0 0" rpy="0 0 0" />
+    <parent link="wrist_2_link" />
+    <child link="robotiq_85_base_link" />
+    <axis xyz="1 0 0" />
+    <limit lower="-3.14159265358979" upper="3.14159265358979" effort="1000" velocity="2.0"/>
+  </joint>
   <link
     name="robotiq_85_base_link">

File: urdf/robot.urdf.xacro (robot description, xacro)
@@ -1,188 +1,188 @@
 <?xml version="1.0"?>
 <robot name="arm" xmlns:xacro="http://www.ros.org/wiki/xacro">
-    <xacro:include filename="gripper.urdf.xacro"/>
-    <material name="grey">
+  <!-- <xacro:include filename="gripper.urdf.xacro"/> -->
+  <material name="grey">
+    <color rgba="0.5 0.5 0.5 1" />
+  </material>
+  <link name="base_link">
+    <visual>
+      <origin xyz="0 0 0" rpy="0 0 0" />
+      <geometry>
+        <box size="0.25 0.25 0.01" />
+      </geometry>
+      <material name="grey">
         <color rgba="0.5 0.5 0.5 1" />
-    </material>
-    <link name="base_link">
-        <visual>
-            <origin xyz="0 0 0" rpy="0 0 0" />
-            <geometry>
-                <box size="0.25 0.25 0.01" />
-            </geometry>
-            <material name="grey">
-                <color rgba="0.5 0.5 0.5 1" />
-            </material>
-        </visual>
-        <collision>
-            <origin xyz="0 0 0" rpy="0 0 0" />
-            <geometry>
-                <box size="0.20 0.20 0.005" />
-            </geometry>
-        </collision>
-    </link>
-    <joint name="base_base_1" type="revolute">
-        <parent link="base_link"/>
-        <child link="base_1"/>
-        <origin xyz="0.0 0 0.005" rpy="0 0 0"/>
-        <axis xyz="0 0 1"/>
-        <limit effort="1000" lower="-3.14" upper="3.14" velocity="10"/>
-    </joint>
-    <link name="base_1">
-        <visual>
-            <origin xyz="0 0 0.075" rpy="0 0 0"/>
-            <geometry>
-                <cylinder radius="0.03" length="0.15"/>
-            </geometry>
-            <material name="grey"/>
-        </visual>
-        <collision>
-            <origin xyz="0 0 0.075" rpy="0 0 0"/>
-            <geometry>
-                <cylinder radius="0.025" length="0.10"/>
-            </geometry>
-        </collision>
-        <inertial>
-            <origin xyz="0 0 0.075" rpy="0 0 0"/>
-            <mass value="1.0"/>
-            <inertia ixx="0.01" ixy="0" ixz="0" iyy="0.01" iyz="0" izz="0.01"/>
-        </inertial>
-    </link>
-    <joint name="base_1_shoulder" type="revolute">
-        <parent link="base_1"/>
-        <child link="shoulder_link"/>
-        <origin xyz="0.0 0 0.135" rpy="0 0 0"/>
-        <axis xyz="1 0 0"/>
-        <limit effort="1000" lower="-1.57" upper="1.57" velocity="10"/>
-    </joint>
-    <link name="shoulder_link">
-        <visual>
-            <origin xyz="0.063 0 0.160" rpy="0 0 0"/>
-            <geometry>
-                <cylinder radius="0.03" length="0.35"/>
-            </geometry>
-            <material name="grey"/>
-        </visual>
-        <collision>
-            <origin xyz="0.063 0 0.160" rpy="0 0 0"/>
-            <geometry>
-                <cylinder radius="0.025" length="0.30"/>
-            </geometry>
-        </collision>
-        <inertial>
-            <origin xyz="0.063 0 0.160" rpy="0 0 0"/>
-            <mass value="1.0"/>
-            <inertia ixx="0.01" ixy="0" ixz="0" iyy="0.01" iyz="0" izz="0.01"/>
-        </inertial>
-    </link>
-    <joint name="shoulder_upper_arm" type="revolute">
-        <parent link="shoulder_link"/>
-        <child link="upper_arm_link"/>
-        <origin xyz="0.0 0 0.32" rpy="0 0 0"/>
-        <axis xyz="1 0 0"/>
-        <limit effort="1000" lower="-1.57" upper="1.57" velocity="10"/>
-    </joint>
-    <link name="upper_arm_link">
-        <visual>
-            <origin xyz="0.0 0 0.160" rpy="0 0 0"/>
-            <geometry>
-                <cylinder radius="0.03" length="0.35"/>
-            </geometry>
-            <material name="grey"/>
-        </visual>
-        <collision>
-            <origin xyz="0.0 0 0.160" rpy="0 0 0"/>
-            <geometry>
-                <cylinder radius="0.025" length="0.30"/>
-            </geometry>
-        </collision>
-        <inertial>
-            <origin xyz="0.0 0 0.160" rpy="0 0 0"/>
-            <mass value="1.0"/>
-            <inertia ixx="0.01" ixy="0" ixz="0" iyy="0.01" iyz="0" izz="0.01"/>
-        </inertial>
-    </link>
-    <joint name="upper_arm_forearm" type="revolute">
-        <parent link="upper_arm_link"/>
-        <child link="forearm_link"/>
-        <origin xyz="0.0 0 0.305" rpy="0 0 0"/>
-        <axis xyz="1 0 0"/>
-        <limit effort="1000" lower="-1.57" upper="1.57" velocity="10"/>
-    </joint>
-    <link name="forearm_link">
-        <visual>
-            <origin xyz="0.068 0 0" rpy="0 1.57 0"/>
-            <geometry>
-                <cylinder radius="0.03" length="0.07"/>
-            </geometry>
-            <material name="grey"/>
-        </visual>
-        <collision>
-            <origin xyz="0.068 0 0" rpy="0 1.57 0"/>
-            <geometry>
-                <cylinder radius="0.025" length="0.06"/>
-            </geometry>
-        </collision>
-        <inertial>
-            <origin xyz="0.068 0 0" rpy="0 1.57 0"/>
-            <mass value="1.0"/>
-            <inertia ixx="0.01" ixy="0" ixz="0" iyy="0.01" iyz="0" izz="0.01"/>
-        </inertial>
-    </link>
-    <joint name="forearm_wrist_1" type="revolute">
-        <parent link="forearm_link"/>
-        <child link="wrist_1_link"/>
-        <origin xyz="0.065 0 0.03" rpy="0 0 0"/>
-        <axis xyz="0.0 0.0 1.0"/>
-        <limit effort="1000" lower="-1.57" upper="1.57" velocity="10"/>
-    </joint>
-    <link name="wrist_1_link">
-        <visual>
-            <origin xyz="0.0 0 0.053" rpy="0 0 0"/>
-            <geometry>
-                <cylinder radius="0.03" length="0.1"/>
-            </geometry>
-            <material name="grey"/>
-        </visual>
-        <collision>
-            <origin xyz="0.0 0 0.053" rpy="0 0 0"/>
-            <geometry>
-                <cylinder radius="0.025" length="0.09"/>
-            </geometry>
-        </collision>
-        <inertial>
-            <origin xyz="0.0 0 0.053" rpy="0 0 0"/>
-            <mass value="1.0"/>
-            <inertia ixx="0.01" ixy="0" ixz="0" iyy="0.01" iyz="0" izz="0.01"/>
-        </inertial>
-    </link>
-    <joint name="wrist_1_wrist_2" type="revolute">
-        <parent link="wrist_1_link"/>
-        <child link="wrist_2_link"/>
-        <origin xyz="0.03 0 0.073" rpy="0 0 0"/>
-        <axis xyz="1 0 0"/>
-        <limit effort="1000" lower="-1.57" upper="1.57" velocity="10"/>
-    </joint>
-    <link name="wrist_2_link">
-        <visual>
-            <origin xyz="0.028 0.0 0.0" rpy="0 1.57 0" />
-            <geometry>
-                <cylinder radius="0.03" length="0.05"/>
-            </geometry>
-            <material name="grey"/>
-        </visual>
-        <collision>
-            <origin xyz="0.028 0.0 0.0" rpy="0 1.57 0" />
-            <geometry>
-                <cylinder radius="0.025" length="0.04"/>
-            </geometry>
-        </collision>
-        <inertial>
-            <origin xyz="0.028 0.0 0.0" rpy="0 1.57 0" />
-            <mass value="1.0"/>
-            <inertia ixx="0.01" ixy="0" ixz="0" iyy="0.01" iyz="0" izz="0.01"/>
-        </inertial>
-    </link>
-    <joint name="wrist_2_end_effector" type="fixed">
+      </material>
+    </visual>
+    <collision>
+      <origin xyz="0 0 0" rpy="0 0 0" />
+      <geometry>
+        <box size="0.20 0.20 0.005" />
+      </geometry>
+    </collision>
+  </link>
+  <joint name="base_base_1" type="revolute">
+    <parent link="base_link"/>
+    <child link="base_1"/>
+    <origin xyz="0.0 0 0.005" rpy="0 0 0"/>
+    <axis xyz="0 0 1"/>
+    <limit effort="1000" lower="-3.14" upper="3.14" velocity="10"/>
+  </joint>
+  <link name="base_1">
+    <visual>
+      <origin xyz="0 0 0.075" rpy="0 0 0"/>
+      <geometry>
+        <cylinder radius="0.03" length="0.15"/>
+      </geometry>
+      <material name="grey"/>
+    </visual>
+    <collision>
+      <origin xyz="0 0 0.075" rpy="0 0 0"/>
+      <geometry>
+        <cylinder radius="0.025" length="0.10"/>
+      </geometry>
+    </collision>
+    <inertial>
+      <origin xyz="0 0 0.075" rpy="0 0 0"/>
+      <mass value="1.0"/>
+      <inertia ixx="0.01" ixy="0" ixz="0" iyy="0.01" iyz="0" izz="0.01"/>
+    </inertial>
+  </link>
+  <joint name="base_1_shoulder" type="revolute">
+    <parent link="base_1"/>
+    <child link="shoulder_link"/>
+    <origin xyz="0.0 0 0.135" rpy="0 0 0"/>
+    <axis xyz="1 0 0"/>
+    <limit effort="1000" lower="-1.57" upper="1.57" velocity="10"/>
+  </joint>
+  <link name="shoulder_link">
+    <visual>
+      <origin xyz="0.063 0 0.160" rpy="0 0 0"/>
+      <geometry>
+        <cylinder radius="0.03" length="0.35"/>
+      </geometry>
+      <material name="grey"/>
+    </visual>
+    <collision>
+      <origin xyz="0.063 0 0.160" rpy="0 0 0"/>
+      <geometry>
+        <cylinder radius="0.025" length="0.30"/>
+      </geometry>
+    </collision>
+    <inertial>
+      <origin xyz="0.063 0 0.160" rpy="0 0 0"/>
+      <mass value="1.0"/>
+      <inertia ixx="0.01" ixy="0" ixz="0" iyy="0.01" iyz="0" izz="0.01"/>
+    </inertial>
+  </link>
+  <joint name="shoulder_upper_arm" type="revolute">
+    <parent link="shoulder_link"/>
+    <child link="upper_arm_link"/>
+    <origin xyz="0.0 0 0.32" rpy="0 0 0"/>
+    <axis xyz="1 0 0"/>
+    <limit effort="1000" lower="-1.57" upper="1.57" velocity="10"/>
+  </joint>
+  <link name="upper_arm_link">
+    <visual>
+      <origin xyz="0.0 0 0.160" rpy="0 0 0"/>
+      <geometry>
+        <cylinder radius="0.03" length="0.35"/>
+      </geometry>
+      <material name="grey"/>
+    </visual>
+    <collision>
+      <origin xyz="0.0 0 0.160" rpy="0 0 0"/>
+      <geometry>
+        <cylinder radius="0.025" length="0.30"/>
+      </geometry>
+    </collision>
+    <inertial>
+      <origin xyz="0.0 0 0.160" rpy="0 0 0"/>
+      <mass value="1.0"/>
+      <inertia ixx="0.01" ixy="0" ixz="0" iyy="0.01" iyz="0" izz="0.01"/>
+    </inertial>
+  </link>
+  <joint name="upper_arm_forearm" type="revolute">
+    <parent link="upper_arm_link"/>
+    <child link="forearm_link"/>
+    <origin xyz="0.0 0 0.305" rpy="0 0 0"/>
+    <axis xyz="1 0 0"/>
+    <limit effort="1000" lower="-1.57" upper="1.57" velocity="10"/>
+  </joint>
+  <link name="forearm_link">
+    <visual>
+      <origin xyz="0.068 0 0" rpy="0 1.57 0"/>
+      <geometry>
+        <cylinder radius="0.03" length="0.07"/>
+      </geometry>
+      <material name="grey"/>
+    </visual>
+    <collision>
+      <origin xyz="0.068 0 0" rpy="0 1.57 0"/>
+      <geometry>
+        <cylinder radius="0.025" length="0.06"/>
+      </geometry>
+    </collision>
+    <inertial>
+      <origin xyz="0.068 0 0" rpy="0 1.57 0"/>
+      <mass value="1.0"/>
+      <inertia ixx="0.01" ixy="0" ixz="0" iyy="0.01" iyz="0" izz="0.01"/>
+    </inertial>
+  </link>
+  <joint name="forearm_wrist_1" type="revolute">
+    <parent link="forearm_link"/>
+    <child link="wrist_1_link"/>
+    <origin xyz="0.065 0 0.03" rpy="0 0 0"/>
+    <axis xyz="0.0 0.0 1.0"/>
+    <limit effort="1000" lower="-1.57" upper="1.57" velocity="10"/>
+  </joint>
+  <link name="wrist_1_link">
+    <visual>
+      <origin xyz="0.0 0 0.053" rpy="0 0 0"/>
+      <geometry>
+        <cylinder radius="0.03" length="0.1"/>
+      </geometry>
+      <material name="grey"/>
+    </visual>
+    <collision>
+      <origin xyz="0.0 0 0.053" rpy="0 0 0"/>
+      <geometry>
+        <cylinder radius="0.025" length="0.09"/>
+      </geometry>
+    </collision>
+    <inertial>
+      <origin xyz="0.0 0 0.053" rpy="0 0 0"/>
+      <mass value="1.0"/>
+      <inertia ixx="0.01" ixy="0" ixz="0" iyy="0.01" iyz="0" izz="0.01"/>
+    </inertial>
+  </link>
+  <joint name="wrist_1_wrist_2" type="revolute">
+    <parent link="wrist_1_link"/>
+    <child link="wrist_2_link"/>
+    <origin xyz="0.03 0 0.073" rpy="0 0 0"/>
+    <axis xyz="1 0 0"/>
+    <limit effort="1000" lower="-1.57" upper="1.57" velocity="10"/>
+  </joint>
+  <link name="wrist_2_link">
+    <visual>
+      <origin xyz="0.028 0.0 0.0" rpy="0 1.57 0" />
+      <geometry>
+        <cylinder radius="0.03" length="0.05"/>
+      </geometry>
+      <material name="grey"/>
+    </visual>
+    <collision>
+      <origin xyz="0.028 0.0 0.0" rpy="0 1.57 0" />
+      <geometry>
+        <cylinder radius="0.025" length="0.04"/>
+      </geometry>
+    </collision>
+    <inertial>
+      <origin xyz="0.028 0.0 0.0" rpy="0 1.57 0" />
+      <mass value="1.0"/>
+      <inertia ixx="0.01" ixy="0" ixz="0" iyy="0.01" iyz="0" izz="0.01"/>
+    </inertial>
+  </link>
+  <!-- <joint name="wrist_2_end_effector" type="fixed">
         <parent link="wrist_2_link"/>
         <child link="end_effector_link"/>
@@ -208,39 +208,558 @@
             <inertia ixx="0.0001" ixy="0" ixz="0" iyy="0.0001" iyz="0" izz="0.0001"/>
         </inertial>
-    </link>
-    <ros2_control name="ArmHardware" type="system">
-      <hardware>
-        <plugin>fake_components/GenericSystem</plugin>
-      </hardware>
-      <joint name="base_base_1">
-        <command_interface name="position"/>
-        <state_interface name="position"/>
-        <state_interface name="velocity"/>
-      </joint>
-      <joint name="base_1_shoulder">
-        <command_interface name="position"/>
-        <state_interface name="position"/>
-        <state_interface name="velocity"/>
-      </joint>
-      <joint name="shoulder_upper_arm">
-        <command_interface name="position"/>
-        <state_interface name="position"/>
-        <state_interface name="velocity"/>
-      </joint>
-      <joint name="upper_arm_forearm">
-        <command_interface name="position"/>
-        <state_interface name="position"/>
-        <state_interface name="velocity"/>
-      </joint>
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