Commit message: started configuring moveit

File: urdf/robot.urdf.xacro (robot description, xacro)
@@ -23,5 +23,5 @@
         <origin xyz="0.0 0 0.0" rpy="0 0 0"/>
         <axis xyz="0 0 1"/>
-        <limit effort="1000" lower="-3.14159265359" upper="3.14159265359" velocity="10"/>
+        <limit effort="1000" lower="-3.14" upper="3.14" velocity="10"/>
     </joint>
     <joint name="base_shoulder" type="revolute">
@@ -30,5 +30,5 @@
         <origin xyz="0.0 0 0.15" rpy="0 0 0"/>
         <axis xyz="1 0 0"/>
-        <limit effort="1000" lower="-3.14159265359" upper="3.14159265359" velocity="10"/>
+        <limit effort="1000" lower="-1.57" upper="1.57" velocity="10"/>
     </joint >
     <joint name="shoulder_upper_arm" type="revolute">
@@ -37,5 +37,5 @@
         <origin xyz="0.0 0 0.34" rpy="0 0 0"/>
         <axis xyz="1 0 0"/>
-        <limit effort="1000" lower="-3.14159265359" upper="3.14159265359" velocity="10"/>
+        <limit effort="1000" lower="-1.57" upper="1.57" velocity="10"/>
     </joint>
     <joint name="upper_arm_forearm" type="revolute">
@@ -44,5 +44,5 @@
         <origin xyz="0.0 0 0.32" rpy="0 0 0"/>
         <axis xyz="1 0 0"/>
-        <limit effort="1000" lower="-3.14159265359" upper="3.14159265359" velocity="10"/>
+        <limit effort="1000" lower="-1.57" upper="1.57" velocity="10"/>
     </joint>
     <joint name="forearm_wrist_1" type="revolute">
@@ -51,5 +51,5 @@
         <origin xyz="0.065 0 0" rpy="0 0 0"/>
         <axis xyz="0.0 0.0 1.0"/>
-        <limit effort="1000" lower="-3.14159265359" upper="3.14159265359" velocity="10"/>
+        <limit effort="1000" lower="-1.57" upper="1.57" velocity="10"/>
     </joint>
     <joint name="wrist_1_wrist_2" type="revolute">
@@ -58,5 +58,10 @@
         <origin xyz="0.0 0 0.10" rpy="0 0 0"/>
         <axis xyz="1 0 0"/>
-        <limit effort="1000" lower="-3.14159265359" upper="3.14159265359" velocity="10"/>
+        <limit effort="1000" lower="-1.57" upper="1.57" velocity="10"/>
+    </joint>
+    <joint name="wrist_2_end_effector" type="fixed">
+        <parent link="wrist_2_link"/>
+        <child link="end_effector_link"/>
+        <origin xyz="0.08 0 0" rpy="0 0 0"/>
     </joint>
     <link name="base_1">
@@ -84,4 +89,10 @@
             </geometry>
         </visual>
+        <collision>
+            <origin xyz="0.06 0 0.175" rpy="0 0 0"/>
+            <geometry>
+                <cylinder radius="0.03" length="0.35"/>
+            </geometry>
+        </collision>
     </link>
     <link name="upper_arm_link">
@@ -96,7 +107,7 @@
         </visual>
         <collision>
-            <origin xyz="0.0 0 0.075" rpy="0 0 0"/>
+            <origin xyz="0.0 0 0.175" rpy="0 0 0"/>
             <geometry>
-                <cylinder radius="0.03" length="0.25"/>
+                <cylinder radius="0.03" length="0.35"/>
             </geometry>
         </collision>
@@ -109,4 +120,10 @@
             </geometry>
         </visual>
+        <collision>
+            <origin xyz="0.065 0 0" rpy="0 1.57 0"/>
+            <geometry>
+                <cylinder radius="0.03" length="0.07"/>
+            </geometry>
+        </collision>
     </link>
     <link name ="wrist_1_link">
@@ -117,4 +134,10 @@
             </geometry>
         </visual>
+        <collision>
+            <origin xyz="0.0 0 0.08" rpy="0 0 0"/>
+            <geometry>
+                <cylinder radius="0.03" length="0.1"/>
+            </geometry>
+        </collision>
     </link>
     <link name="wrist_2_link" >
@@ -125,4 +148,24 @@
         </geometry>
         </visual>
+        <collision>
+            <origin xyz="0.055 0.0 0.0" rpy="0 1.57 0" />
+            <geometry>
+                <cylinder radius="0.03" length="0.05"/>
+            </geometry>
+        </collision>
+    </link>
+    <link name="end_effector_link">
+        <visual>
+            <origin xyz="0.01 0 0" rpy="0 0 0" />
+            <geometry>
+                <box size="0.1 0.01 0.01"/>
+            </geometry>
+        </visual>
+        <collision>
+            <origin xyz="0.01 0 0" rpy="0 0 0" />
+            <geometry>
+                <box size="0.1 0.01 0.01"/>
+            </geometry>
+        </collision>
     </link>
 </robot>

Commit message: added inertial and collision elements in urdf file

File: urdf/robot.urdf.xacro (robot description, xacro)
@@ -81,4 +81,9 @@
             </geometry>
         </collision>
+        <inertial>
+            <origin xyz="0 0 0.08" rpy="0 0 0"/>
+            <mass value="1.0"/>
+            <inertia ixx="0.01" ixy="0" ixz="0" iyy="0.01" iyz="0" izz="0.01"/>
+        </inertial>
     </link>
     <link name="shoulder_link">
@@ -95,4 +100,9 @@
             </geometry>
         </collision>
+        <inertial>
+            <origin xyz="0.06 0 0.175" rpy="0 0 0"/>
+            <mass value="1.0"/>
+            <inertia ixx="0.01" ixy="0" ixz="0" iyy="0.01" iyz="0" izz="0.01"/>
+        </inertial>
     </link>
     <link name="upper_arm_link">
@@ -112,4 +122,9 @@
             </geometry>
         </collision>
+        <inertial>
+            <origin xyz="0.0 0 0.175" rpy="0 0 0"/>
+            <mass value="1.0"/>
+            <inertia ixx="0.01" ixy="0" ixz="0" iyy="0.01" iyz="0" izz="0.01"/>
+        </inertial>
     </link>
     <link name="forearm_link">
@@ -126,4 +141,9 @@
             </geometry>
         </collision>
+        <inertial>
+            <origin xyz="0.065 0 0" rpy="0 1.57 0"/>
+            <mass value="1.0"/>
+            <inertia ixx="0.01" ixy="0" ixz="0" iyy="0.01" iyz="0" izz="0.01"/>
+        </inertial>
     </link>
     <link name ="wrist_1_link">
@@ -140,18 +160,28 @@
             </geometry>
         </collision>
+        <inertial>
+            <origin xyz="0.0 0 0.08" rpy="0 0 0"/>
+            <mass value="1.0"/>
+            <inertia ixx="0.01" ixy="0" ixz="0" iyy="0.01" iyz="0" izz="0.01"/>
+        </inertial>
     </link>
     <link name="wrist_2_link" >
         <visual>
             <origin xyz="0.055 0.0 0.0" rpy="0 1.57 0" />
-        <geometry>
-            <cylinder radius="0.03" length="0.05"/>
-        </geometry>
-        </visual>
-        <collision>
-            <origin xyz="0.055 0.0 0.0" rpy="0 1.57 0" />
             <geometry>
                 <cylinder radius="0.03" length="0.05"/>
             </geometry>
-        </collision>
+            <collision>
+                <origin xyz="0.055 0.0 0.0" rpy="0 1.57 0" />
+                <geometry>
+                    <cylinder radius="0.03" length="0.05"/>
+                </geometry>
+            </collision>
+            <inertial>
+                <origin xyz="0.055 0.0 0.0" rpy="0 1.57 0" />
+                <mass value="1.0"/>
+                <inertia ixx="0.01" ixy="0" ixz="0" iyy="0.01" iyz="0" izz="0.01"/>
+            </inertial>
+        </visual>
     </link>
     <link name="end_effector_link">

Commit message: now gripper is working and added gazebo to launch file

File: urdf/robot.urdf.xacro (robot description, xacro)
@@ -1,5 +1,10 @@
 <?xml version="1.0"?>
 <robot name="arm" xmlns:xacro="http://www.ros.org/wiki/xacro">
-  <!-- <xacro:include filename="gripper.urdf.xacro"/> -->
+  <xacro:include filename="camera.urdf.xacro"/>
+  <joint name="camera_end_effector" type="fixed">
+    <parent link="wrist_2_link"/>
+    <child link="camera_link"/>
+    <origin xyz="0.047 0.050 0" rpy="0 0 0" />
+  </joint>
   <material name="grey">
     <color rgba="0.5 0.5 0.5 1" />
@@ -18,5 +23,5 @@
       <origin xyz="0 0 0" rpy="0 0 0" />
       <geometry>
-        <box size="0.20 0.20 0.005" />
+        <box size="0.25 0.25 0.01" />
       </geometry>
     </collision>
@@ -40,5 +45,5 @@
       <origin xyz="0 0 0.075" rpy="0 0 0"/>
       <geometry>
-        <cylinder radius="0.025" length="0.10"/>
+        <cylinder radius="0.03" length="0.15"/>
       </geometry>
     </collision>
@@ -67,5 +72,5 @@
       <origin xyz="0.063 0 0.160" rpy="0 0 0"/>
       <geometry>
-        <cylinder radius="0.025" length="0.30"/>
+        <cylinder radius="0.03" length="0.35"/>
       </geometry>
     </collision>
@@ -94,5 +99,5 @@
       <origin xyz="0.0 0 0.160" rpy="0 0 0"/>
       <geometry>
-        <cylinder radius="0.025" length="0.30"/>
+        <cylinder radius="0.03" length="0.35"/>
       </geometry>
     </collision>
@@ -121,5 +126,5 @@
       <origin xyz="0.068 0 0" rpy="0 1.57 0"/>
       <geometry>
-        <cylinder radius="0.025" length="0.06"/>
+        <cylinder radius="0.03" length="0.07"/>
       </geometry>
     </collision>
@@ -148,5 +153,5 @@
       <origin xyz="0.0 0 0.053" rpy="0 0 0"/>
       <geometry>
-        <cylinder radius="0.025" length="0.09"/>
+        <cylinder radius="0.03" length="0.1"/>
       </geometry>
     </collision>
@@ -175,5 +180,5 @@
       <origin xyz="0.028 0.0 0.0" rpy="0 1.57 0" />
       <geometry>
-        <cylinder radius="0.025" length="0.04"/>
+        <cylinder radius="0.03" length="0.05"/>
       </geometry>
     </collision>
@@ -762,4 +767,9 @@
       <state_interface name="velocity"/>
     </joint>
+    <joint name="finger_joint">
+      <command_interface name="position"/>
+      <state_interface name="position"/>
+      <state_interface name="velocity"/>
+    </joint>
   </ros2_control>
 </robot>

Commit message: reconnecting

File: urdf/robot.urdf.xacro (robot description, xacro)
@@ -26,4 +26,9 @@
       </geometry>
     </collision>
+    <inertial>
+      <origin xyz="0 0 0" rpy="0 0 0"/>
+      <mass value="1.0"/>
+      <inertia ixx="0.01" ixy="0" ixz="0" iyy="0.01" iyz="0" izz="0.01"/>
+    </inertial>
   </link>
   <joint name="base_base_1" type="revolute">
@@ -494,103 +499,93 @@
         offset="0" />
   </joint>
-  <link
-      name="right_inner_knuckle">
-    <inertial>
-      <origin
-          xyz="0.0168606186773776 3.93808471820465E-10 0.0226699950793434"
-          rpy="0 0 0" />
-      <mass
-          value="0.0110930853895903" />
-      <inertia
-          ixx="4.27134775939882E-06"
-          ixy="-8.53568456728898E-15"
-          ixz="1.77774229944246E-06"
-          iyy="3.96548790524392E-06"
-          iyz="-8.45108024914164E-15"
-          izz="3.20325997634666E-06" />
-    </inertial>
-    <visual>
-      <origin
-          xyz="0 0 0"
-          rpy="0 0 0" />
-      <geometry>
-        <mesh
-            filename="package://robotic_manipulator_6_dof/meshes/inner_knuckle_fine.STL" />
-      </geometry>
-      <material
-          name="">
-        <color
-            rgba="0.1 0.1 0.1 1" />
-      </material>
-    </visual>
-    <collision>
-      <origin
-          xyz="0 0 0"
-          rpy="0 0 0" />
-      <geometry>
-        <mesh
-            filename="package://robotic_manipulator_6_dof/meshes/inner_knuckle_coarse.STL" />
-      </geometry>
-    </collision>
-  </link>
-  <joint
-      name="right_inner_knuckle_joint"
-      type="revolute">
+  <link name="right_inner_knuckle">
+    <inertial>
+      <origin
+        xyz="0.0168606186773776 3.93808471820465E-10 0.0226699950793434"
+        rpy="0 0 0" />
+      <mass
+        value="0.0110930853895903" />
+      <inertia
+        ixx="4.27134775939882E-06"
+        ixy="-8.53568456728898E-15"
+        ixz="1.77774229944246E-06"
+        iyy="3.96548790524392E-06"
+        iyz="-8.45108024914164E-15"
+        izz="3.20325997634666E-06"/>
+    </inertial>
+    <visual>
+      <origin
+        xyz="0 0 0"
+        rpy="0 0 0" />
+      <geometry>
+        <mesh filename="package://robotic_manipulator_6_dof/meshes/inner_knuckle_fine.STL" />
+      </geometry>
+      <material name="">
+        <color rgba="0.1 0.1 0.1 1" />
+      </material>
+    </visual>
+    <collision>
+      <origin
+        xyz="0 0 0"
+        rpy="0 0 0" />
+      <geometry>
+        <mesh filename="package://robotic_manipulator_6_dof/meshes/inner_knuckle_coarse.STL" />
+      </geometry>
+    </collision>
+  </link>
+  <joint name="right_inner_knuckle_joint" type="revolute">
     <origin
-        xyz="-0.0126999999998499 0 0.0693075000000361"
-        rpy="0 0 3.14159265358979" />
+      xyz="-0.0126999999998499 0 0.0693075000000361"
+      rpy="0 0 3.14159265358979" />
     <parent
-        link="robotiq_85_base_link" />
+      link="robotiq_85_base_link" />
     <child
-        link="right_inner_knuckle" />
+      link="right_inner_knuckle" />
     <axis
-        xyz="0 1 0" />
+      xyz="0 1 0" />
     <limit
-        lower="0"
-        upper="0.8757"
-        velocity="2.0"
-        effort="1000" />
+      lower="0"
+      upper="0.8757"
+      velocity="2.0"
+      effort="1000" />
     <mimic
-        joint="finger_joint"
-        multiplier="-1"
-        offset="0" />
-  </joint>
-  <link
-      name="right_inner_finger">
-    <inertial>
-      <origin
-          xyz="0.00602756228812038 -6.47284509480176E-15 0.00669925609578108"
-          rpy="0 0 0" />
-      <mass
-          value="0.00724255346165744" />
-      <inertia
-          ixx="1.47824283625957E-06"
-          ixy="-3.95952064019123E-19"
-          ixz="-3.45268708875543E-07"
-          iyy="1.70064480838394E-06"
-          iyz="3.55286507960029E-19"
-          izz="4.77151241114822E-07" />
-    </inertial>
-    <visual>
-      <origin
-          xyz="0 0 0"
-          rpy="0 0 0" />
-      <geometry>
-        <mesh
-            filename="package://robotic_manipulator_6_dof/meshes/inner_finger_fine.STL" />
-      </geometry>
-      <material
-          name="">
-        <color
-            rgba="0.1 0.1 0.1 1" />
-      </material>
-    </visual>
-    <collision>
-      <origin
-          xyz="0 0 0"
-          rpy="0 0 0" />
-      <geometry>
-        <mesh
-            filename="package://robotic_manipulator_6_dof/meshes/inner_finger_coarse.STL" />
+      joint="finger_joint"
+      multiplier="-1"
+      offset="0" />
+  </joint>
+  <link name="right_inner_finger">
+    <inertial>
+      <origin
+        xyz="0.00602756228812038 -6.47284509480176E-15 0.00669925609578108"
+        rpy="0 0 0" />
+      <mass
+        value="0.00724255346165744" />
+      <inertia
+        ixx="1.47824283625957E-06"
+        ixy="-3.95952064019123E-19"
+        ixz="-3.45268708875543E-07"
+        iyy="1.70064480838394E-06"
+        iyz="3.55286507960029E-19"
+        izz="4.77151241114822E-07" />
+    </inertial>
+    <visual>
+      <origin
+        xyz="0 0 0"
+        rpy="0 0 0" />
+      <geometry>
+        <mesh
+          filename="package://robotic_manipulator_6_dof/meshes/inner_finger_fine.STL" />
+      </geometry>
+      <material name="">
+        <color rgba="0.1 0.1 0.1 1" />
+      </material>
+    </visual>
+    <collision>
+      <origin
+        xyz="0 0 0"
+        rpy="0 0 0" />
+      <geometry>
+        <mesh
+          filename="package://robotic_manipulator_6_dof/meshes/inner_finger_coarse.STL" />
       </geometry>
     </collision>
@@ -600,21 +595,21 @@
       type="revolute">
     <origin
-        xyz="0.0341060475457406 0 0.0458573878541688"
-        rpy="0 0 0" />
+      xyz="0.0341060475457406 0 0.0458573878541688"
+      rpy="0 0 0" />
     <parent
-        link="right_inner_knuckle" />
+      link="right_inner_knuckle" />
     <child
-        link="right_inner_finger" />
+      link="right_inner_finger" />
     <axis
-        xyz="0 1 0" />
+      xyz="0 1 0" />
     <limit
-        lower="0"
-        upper="0.8757"
-        velocity="2.0"
-        effort="1000" />
+      lower="0"
+      upper="0.8757"
+      velocity="2.0"
+      effort="1000" />
     <mimic
-        joint="finger_joint"
-        multiplier="1"
-        offset="0" />
+      joint="finger_joint"
+      multiplier="1"
+      offset="0" />
   </joint>
   <link
@@ -622,8 +617,8 @@
     <inertial>
       <origin
-          xyz="0.0178097074051638 3.60493211424024E-11 0.00233123458346721"
-          rpy="0 0 0" />
-      <mass
-          value="0.00684838849401352" />
+        xyz="0.0178097074051638 3.60493211424024E-11 0.00233123458346721"
+        rpy="0 0 0" />
+      <mass
+        value="0.00684838849401352" />
       <inertia
           ixx="2.70004361573169E-07"
@@ -636,14 +631,14 @@
     <visual>
       <origin
-          xyz="0 0 0"
-          rpy="0 0 0" />
-      <geometry>
-        <mesh
-            filename="package://robotic_manipulator_6_dof/meshes/outer_knuckle_fine.STL" />
+        xyz="0 0 0"
+        rpy="0 0 0" />
+      <geometry>
+        <mesh
+          filename="package://robotic_manipulator_6_dof/meshes/outer_knuckle_fine.STL" />
       </geometry>
       <material
           name="">
         <color
-            rgba="0.1 0.1 0.1 1" />
+          rgba="0.1 0.1 0.1 1" />
       </material>
     </visual>
@@ -735,5 +730,5 @@
   <ros2_control name="ArmHardware" type="system">
     <hardware>
-      <plugin>fake_components/GenericSystem</plugin>
+      <plugin>gazebo_ros2_control/GazeboSystem</plugin>
     </hardware>
     <joint name="base_base_1">
@@ -773,3 +768,10 @@
     </joint>
   </ros2_control>
+  <gazebo>
+    <plugin filename="gz_ros2_control-system" name="gz_ros2_control::GazeboSimROS2ControlPlugin">
+      <robot_param>robot_description</robot_param>
+      <robot_param_node>robot_state_publisher</robot_param_node>
+      <parameters>$(find robotic_manipulator_6_dof)/config/ros2_controllers.yaml</parameters>
+    </plugin>
+  </gazebo>
 </robot>

Commit message: did some minute changes

File: urdf/robot.urdf.xacro (robot description, xacro)
@@ -28,5 +28,5 @@
     <inertial>
       <origin xyz="0 0 0" rpy="0 0 0"/>
-      <mass value="1.0"/>
+      <mass value="100.0"/>
       <inertia ixx="0.01" ixy="0" ixz="0" iyy="0.01" iyz="0" izz="0.01"/>
     </inertial>
@@ -730,5 +730,5 @@
   <ros2_control name="ArmHardware" type="system">
     <hardware>
-      <plugin>gazebo_ros2_control/GazeboSystem</plugin>
+      <plugin>gz_ros2_control/GazeboSimSystem</plugin>
     </hardware>
     <joint name="base_base_1">
@@ -769,8 +769,9 @@
   </ros2_control>
   <gazebo>
-    <plugin filename="gz_ros2_control-system" name="gz_ros2_control::GazeboSimROS2ControlPlugin">
+    <plugin filename="libgz_ros2_control-system.so" name="gz_ros2_control::GazeboSimROS2ControlPlugin">
       <robot_param>robot_description</robot_param>
       <robot_param_node>robot_state_publisher</robot_param_node>
-      <parameters>$(find robotic_manipulator_6_dof)/config/ros2_controllers.yaml</parameters>
+      <parameters>$(find move_it_config)/config/ros2_controllers.yaml</parameters>
+      <controller_manager_name>controller_manager</controller_manager_name>
     </plugin>
   </gazebo>
