Commit message: did changes according to load gazebo

File: urdf/camera.urdf.xacro (robot description, xacro)
@@ -34,8 +34,26 @@
           </image>
           <clip>
-            <near>0.1</near>
-            <far>100</far>
+            <near>0.05</near>
+            <far>5.0</far>
           </clip>
         </camera>
+        <plugin name="camera_controller" filename="libgazebo_ros_camera.so">
+          <alwaysOn>true</alwaysOn>
+          <updateRate>30.0</updateRate>
+          <cameraName>camera</cameraName>
+          <frameName>camera_link</frameName>
+          <imageTopicName>rgb/image_raw</imageTopicName>
+          <cameraInfoTopicName>rgb/camera_info</cameraInfoTopicName>
+          <depthImageTopicName>depth/image_raw</depthImageTopicName>
+          <depthImageCameraInfoTopicName>depth/camera_info</depthImageCameraInfoTopicName>
+          <pointCloudTopicName>depth/points</pointCloudTopicName>
+          <pointCloudCutoff>0.5</pointCloudCutoff>
+          <pointCloudCutoffMax>5.0</pointCloudCutoffMax>
+          <distortionK1>0.0</distortionK1>
+          <distortionK2>0.0</distortionK2>
+          <distortionK3>0.0</distortionK3>
+          <distortionT1>0.0</distortionT1>
+          <distortionT2>0.0</distortionT2>
+        </plugin>
       </sensor>
     </gazebo>

File: urdf/robot.urdf.xacro (robot description, xacro)
@@ -1,4 +1,16 @@
 <?xml version="1.0"?>
 <robot name="arm" xmlns:xacro="http://www.ros.org/wiki/xacro">
+  <xacro:macro name="control" params="joint">
+    <transmission name="${joint}_transmission">
+      <type>transmission_interface/SimpleTransmission</type>
+      <joint name="${joint}">
+        <hardwareInterface>hardware_interface/EffortJointInterface</hardwareInterface>
+      </joint>
+      <actuator name="${joint}_motor">
+        <mechanicalReduction>1.0</mechanicalReduction>
+        <hardwareInterface>hardware_interface/EffortJointInterface</hardwareInterface>
+      </actuator>
+    </transmission>
+  </xacro:macro>
   <xacro:include filename="camera.urdf.xacro"/>
   <joint name="camera_end_effector" type="fixed">
@@ -195,28 +207,35 @@
   </link>
   <!-- <joint name="wrist_2_end_effector" type="fixed">
-        <parent link="wrist_2_link"/>
-        <child link="end_effector_link"/>
-        <origin xyz="0.061 0 0" rpy="0 0 0"/>
+    <parent link="wrist_2_link"/>
+    <child link="end_effector_link"/>
+    <origin xyz="0.061 0 0" rpy="0 0 0"/>
     </joint>
     <link name="end_effector_link">
-        <visual>
+      <visual>
+        <origin xyz="0 0 0" rpy="0 0 0" />
+        <geometry>
+          <box size="0.01 0.01 0.01"/>
+          </geometry>
+          <material name="grey"/>
+          </visual>
+          <collision>
             <origin xyz="0 0 0" rpy="0 0 0" />
             <geometry>
-                <box size="0.01 0.01 0.01"/>
-            </geometry>
-            <material name="grey"/>
-        </visual>
-        <collision>
-            <origin xyz="0 0 0" rpy="0 0 0" />
-            <geometry>
-                <box size="0.005 0.005 0.005"/>
-            </geometry>
-        </collision>
-        <inertial>
-            <origin xyz="0 0 0" rpy="0 0 0"/>
-            <mass value="0.1"/>
-            <inertia ixx="0.0001" ixy="0" ixz="0" iyy="0.0001" iyz="0" izz="0.0001"/>
-        </inertial>
-    </link> -->
+              <box size="0.005 0.005 0.005"/>
+              </geometry>
+              </collision>
+              <inertial>
+                <origin xyz="0 0 0" rpy="0 0 0"/>
+                <mass value="0.1"/>
+                <inertia ixx="0.0001" ixy="0" ixz="0" iyy="0.0001" iyz="0" izz="0.0001"/>
+              </inertial>
+                </link> -->
+  <xacro:control joint="base_base_1"/>
+  <xacro:control joint="base_1_shoulder"/>
+  <xacro:control joint="shoulder_upper_arm"/>
+  <xacro:control joint="upper_arm_forearm"/>
+  <xacro:control joint="forearm_wrist_1"/>
+  <xacro:control joint="wrist_1_wrist_2"/>
+  <xacro:control joint="finger_joint"/>
   <joint name="wrist_2_end_effector" type="fixed">
     <origin xyz="0.061 0 0" rpy="0 1.57 0" />
@@ -225,69 +244,69 @@
   </joint>
   <link
-      name="robotiq_85_base_link">
-    <inertial>
-      <origin
-          xyz="0 0 0"
-          rpy="0 0 0" />
-      <mass
-          value="0.30915" />
-      <inertia
-          ixx="0.00028972"
-          ixy="-5.7879E-10"
-          ixz="-1.8543E-06"
-          iyy="0.00030737"
-          iyz="1.682E-12"
-          izz="0.00019914" />
-    </inertial>
-    <visual>
-      <origin
-          xyz="0 0 0"
-          rpy="0 0 0" />
-      <geometry>
-        <mesh
-            filename="package://robotic_manipulator_6_dof/meshes/robotiq_85_base_link_fine.STL" />
+  name="robotiq_85_base_link">
+  <inertial>
+    <origin
+    xyz="0 0 0"
+    rpy="0 0 0" />
+    <mass
+    value="0.30915" />
+    <inertia
+    ixx="0.00028972"
+    ixy="-5.7879E-10"
+    ixz="-1.8543E-06"
+    iyy="0.00030737"
+    iyz="1.682E-12"
+    izz="0.00019914" />
+  </inertial>
+  <visual>
+    <origin
+    xyz="0 0 0"
+    rpy="0 0 0" />
+    <geometry>
+      <mesh
+      filename="package://robotic_manipulator_6_dof/meshes/robotiq_85_base_link_fine.STL" />
+    </geometry>
+    <material
+      name="">
+      <color
+      rgba="0.1 0.1 0.1 1" />
+    </material>
+  </visual>
+  <collision>
+    <origin
+    xyz="0 0 0"
+    rpy="0 0 0" />
+    <geometry>
+      <mesh
+      filename="package://robotic_manipulator_6_dof/meshes/robotiq_85_base_link_coarse.STL" />
+    </geometry>
+  </collision>
+</link>
+<link
+name="left_outer_knuckle">
+<inertial>
+  <origin
+  xyz="0.0178331863169983 3.68915177224286E-11 0.0021442477325704"
+  rpy="0 0 0" />
+  <mass
+  value="0.00684838849434396" />
+  <inertia
+  ixx="2.66832029033166E-07"
+  ixy="1.66142314639824E-15"
+  ixz="1.45945633322873E-07"
+  iyy="1.3889233257419E-06"
+  iyz="2.82951161241588E-15"
+  izz="1.26603336914415E-06" />
+</inertial>
+    <visual>
+      <origin
+      xyz="0 0 0"
+      rpy="0 0 0" />
+      <geometry>
+        <mesh
+        filename="package://robotic_manipulator_6_dof/meshes/outer_knuckle_fine.STL" />
       </geometry>
       <material
-          name="">
-        <color
-            rgba="0.1 0.1 0.1 1" />
-      </material>
-    </visual>
-    <collision>
-      <origin
-          xyz="0 0 0"
-          rpy="0 0 0" />
-      <geometry>
-        <mesh
-            filename="package://robotic_manipulator_6_dof/meshes/robotiq_85_base_link_coarse.STL" />
-      </geometry>
-    </collision>
-  </link>
-  <link
-      name="left_outer_knuckle">
-    <inertial>
-      <origin
-          xyz="0.0178331863169983 3.68915177224286E-11 0.0021442477325704"
-          rpy="0 0 0" />
-      <mass
-          value="0.00684838849434396" />
-      <inertia
-          ixx="2.66832029033166E-07"
-          ixy="1.66142314639824E-15"
-          ixz="1.45945633322873E-07"
-          iyy="1.3889233257419E-06"
-          iyz="2.82951161241588E-15"
-          izz="1.26603336914415E-06" />
-    </inertial>
-    <visual>
-      <origin
-          xyz="0 0 0"
-          rpy="0 0 0" />
-      <geometry>
-        <mesh
-            filename="package://robotic_manipulator_6_dof/meshes/outer_knuckle_fine.STL" />
-      </geometry>
-      <material
-          name="">
+      name="">
         <color
             rgba="0.1 0.1 0.1 1" />
@@ -730,5 +749,5 @@
   <ros2_control name="ArmHardware" type="system">
     <hardware>
-      <plugin>gz_ros2_control/GzSystem</plugin>
+      <plugin>gz_ros2_control/GazeboSimSystem</plugin>
     </hardware>
     <joint name="base_base_1">
@@ -768,11 +787,21 @@
     </joint>
   </ros2_control>
-  <!-- <gazebo>
+  <gazebo>
     <plugin filename="libgz_ros2_control-system.so" name="gz_ros2_control::GazeboSimROS2ControlPlugin">
       <robot_param>robot_description</robot_param>
       <robot_param_node>robot_state_publisher</robot_param_node>
-      <parameters>robotic_manipulator_6_dof/config/ros2_controllers.yaml</parameters>
+      <parameters>$(find move_it_config)/config/ros2_controllers.yaml</parameters>
       <controller_manager_name>controller_manager</controller_manager_name>
-    </plugin> -->
-  <!-- </gazebo> -->
+    </plugin>
+    <plugin name="gazebo_ros_joint_state_publisher" filename="libgazebo_ros_joint_state_publisher.so">
+      <update_rate>50</update_rate>
+      <joint_name>base_base_1</joint_name>
+      <joint_name>base_1_shoulder</joint_name>
+      <joint_name>shoulder_upper_arm</joint_name>
+      <joint_name>upper_arm_forearm</joint_name>
+      <joint_name>forearm_wrist_1</joint_name>
+      <joint_name>wrist_1_wrist_2</joint_name>
+      <joint_name>finger_joint</joint_name>
+    </plugin>
+  </gazebo>
 </robot>
